Commit message: system visualisation beginnings

File: sorter_ws/src/robot_description/urdf/end_effector.urdf (robot description, URDF)
Before this commit: robot parallel_gripper_end_effector, 6 links, 5 joints
Links:
- removed link wrist_3_link
- added link end_effector_mount_connector; collision mesh filename=package://robot_description/meshes/end_effector_mount_conne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 scale=0.001 0.001 0.001; visual mesh filename=package://robot_description/meshes/end_effector_mount_conne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 scale=0.001 0.001 0.001
- link end_effector_main_frame: geometry collision mesh filename=package://robot_description/meshes/end_effector_main_frame.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 scale=0.001 0.001 0.001; visual mesh filename=package://robot_description/meshes/end_effector_main_frame.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 scale=0.001 0.001 0.001
- link gripper_finger_left: geometry collision mesh filename=package://robot_description/meshes/gripper_finger_left.stl scale=0.001 0.001 0.001; visual mesh filename=package://robot_description/meshes/gripper_finger_left.stl scale=0.001 0.001 0.001
- link gripper_finger_right: geometry collision mesh filename=package://robot_description/meshes/gripper_finger_right.stl scale=0.001 0.001 0.001; visual mesh filename=package://robot_description/meshes/gripper_finger_right.stl scale=0.001 0.001 0.001
- link slider_rod_lower: geometry visual mesh filename=package://robot_description/meshes/slider_rod.stl scale=0.001 0.001 0.001
- link slider_rod_upper: geometry visual mesh filename=package://robot_description/meshes/slider_rod.stl scale=0.001 0.001 0.001
Joints:
- removed joint mount_frame_joint
- added joint end_effector_mount_connector_joint: type fixed, parent end_effector_mount_connector, child end_effector_main_frame, origin xyz=0 0.0525 -0.03 rpy=0 0 3.14
- joint frame_slider_lower_joint: origin xyz=0 36 10.5 rpy=0 0 0 -> xyz=0 0.036 0.0105 rpy=0 0 0
- joint frame_slider_upper_joint: origin xyz=0 36 40.5 rpy=0 0 0 -> xyz=0 0.036 0.0405 rpy=0 0 0
- joint left_finger_slide: axis -1 0 0 -> (none); limit lower=0 upper=29 effort=50 velocity=5 -> (none); origin xyz=29 -76 -40 rpy=0 0 0 -> xyz=0.029 -0.076 -0.040 rpy=0 0 0; type prismatic -> fixed
- joint right_finger_slide: axis 1 0 0 -> (none); limit lower=0 upper=29 effort=50 velocity=5 -> (none); origin xyz=-29 -76 -40 rpy=0 0 0 -> xyz=-0.029 -0.076 -0.040 rpy=0 0 0; type prismatic -> fixed
