Commit message: added collision to ee, master launch

File: sorter_ws/src/robot_description/urdf/end_effector.urdf.xacro (robot description, xacro)
@@ -79,4 +79,9 @@
 			<material name='dark_grey'/>
 		</visual>
+		<collision>
+			<geometry>
+				<mesh filename="package://robot_description/meshes/gripper_finger_left.stl" scale="0.001 0.001 0.001"/>
+			</geometry>
+		</collision>
 	</link>
 	<!-- slider rod lower -->
@@ -88,4 +93,9 @@
 			<material name='dark_grey'/>
 		</visual>
+		<collision>
+			<geometry>
+				<mesh filename="package://robot_description/meshes/gripper_finger_left.stl" scale="0.001 0.001 0.001"/>
+			</geometry>
+		</collision>
 	</link>
 	<!--///////////////////////////////////////

Commit message: post wednesday testing

File: sorter_ws/src/robot_description/urdf/end_effector.urdf.xacro (robot description, xacro)
@@ -79,9 +79,9 @@
 			<material name='dark_grey'/>
 		</visual>
-		<collision>
+		<!-- <collision>
 			<geometry>
 				<mesh filename="package://robot_description/meshes/gripper_finger_left.stl" scale="0.001 0.001 0.001"/>
 			</geometry>
-		</collision>
+		</collision>	 -->
 	</link>
 	<!-- slider rod lower -->
@@ -93,9 +93,9 @@
 			<material name='dark_grey'/>
 		</visual>
-		<collision>
+		<!-- <collision>
 			<geometry>
 				<mesh filename="package://robot_description/meshes/gripper_finger_left.stl" scale="0.001 0.001 0.001"/>
 			</geometry>
-		</collision>
+		</collision>	 -->
 	</link>
 	<!--///////////////////////////////////////

File: sorter_ws/src/robot_description/urdf/ur_with_end_effector.xacro (robot description, xacro)
@@ -11,5 +11,5 @@
     <parent link="wrist_3_link"/>
     <child link="end_effector_mount_connector"/>
-    <origin xyz="0 0 0.005" rpy="1.57 0 0"/>
+    <origin xyz="0 0 0.01" rpy="1.57 0 0"/>
   </joint>
 </robot>
